File: MegaBlaster2.kicad_pcb (KiCad board)
At the start: 4 copper layers, 99 x 99 mm, 114 parts, among them J1 USB_B, J2 SWD, J3 Micro_SD_Card, J4 AudioJack3, SW1 SW_SPDT, SW2 SW_Push_Dual, SW3 SW_Push_Dual, SW4 SW_Push_Dual, SW5 SW_Push_Dual, SW6 SW_Push_Dual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

Commit message: Routing
Parts:
- added TP6: TestPoint, TestPoint:TestPoint_Pad_2.0x2.0mm, F.Cu at (194.4, 83.3)
- moved C20 139.3 mm to (102.0, 84.6), turned to 180 degrees
- moved C15 128.8 mm to (102.2, 78.3), turned to 180 degrees
- moved C25 128.4 mm to (144.6, 137.2), turned to 180 degrees
- moved C16 84.7 mm to (153.9, 84.8)
- moved C26 72.4 mm to (164.6, 84.3)
- moved C27 70.9 mm to (166.9, 92.7)
- moved C21 63.1 mm to (149.4, 79.2), turned to 180 degrees
- moved C17 43.2 mm to (140.7, 80.8)
- moved C22 41.2 mm to (143.5, 86.9)
- moved Y2 35.2 mm to (136.4, 83.8), turned to 270 degrees
- moved U6 35.1 mm to (142.0, 83.8)
- moved R2 33.3 mm to (135.1, 79.5)
- moved J2 24.5 mm to (131.2, 81.5)
- moved C19 21.0 mm to (108.0, 112.0), turned to 315 degrees
- moved C11 20.2 mm to (137.0, 92.8), turned to 45 degrees
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Connections:
- U1 pad 16: Net-(U1-Pad16) -> RAM_CS
- U1 pad 35: D0 -> D7
- U1 pad 36: D1 -> D6
- U1 pad 37: D2 -> D5
- U1 pad 38: D3 -> D4
- U1 pad 40: Net-(U1-Pad40) -> PSG_WE
- U1 pad 41: D4 -> D3
- U1 pad 42: D5 -> D2
- U1 pad 43: D6 -> D1
- U1 pad 44: D7 -> D0
- U1 pad 60: RAM_CS -> Net-(U1-Pad60)
Routing:
- net +3V3: track 0.00 -> 239.8 mm, vias 0 -> 6
- net VBOOST: track 0.00 -> 83.2 mm, vias 0 -> 18
- net +5VA: track 0.00 -> 76.5 mm, vias 0 -> 2
- net SDA: track 0.00 -> 69.4 mm, vias 0 -> 2
- net SCL: track 0.00 -> 68.5 mm, vias 0 -> 2
- net D6: track 0.00 -> 62.2 mm, vias 0 -> 1
- net D5: track 0.00 -> 61.8 mm, vias 0 -> 2
- net YM_A1: track 0.00 -> 57.5 mm, vias 0 -> 5
- net YM_A0: track 0.00 -> 57.1 mm, vias 0 -> 3
- net D7: track 0.00 -> 57.0 mm, vias 0 -> 2
- net D+: track 0.00 -> 56.6 mm, vias 0 -> 2
- net PSG_WE: track 0.00 -> 56.5 mm, vias 0 -> 4
- net D-: track 0.00 -> 55.8 mm, vias 0 -> 2
- net PSG_CLK: track 0.00 -> 53.4 mm, vias 0 -> 2
- net D4: track 0.00 -> 53.1 mm, vias 0 -> 2
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- added copper zone on F.Cu, net GND
- added copper zone on F.Cu, net Net-(D1-Pad2)
- added copper zone on F.Cu, net VBOOST
- added copper zone on F.Cu, net VBUS
Other:
- net class THICC added: clearance 0.2, trace_width 1, via_dia 1, via_drill 0.4
- board text added: "*!"

Commit message: Board v1 complete
Parts:
- removed R23, R24: 10R, Resistor_SMD:R_0805_2012Metric
- removed SW1: SW_SPDT, Button_Switch_THT:SW_Slide_1P2T_CK_OS102011MS2Q
- added G***: LOGO, Art:logo_2, F.Cu at (93.5, 109.2)
- added G***: LOGO, Art:logo1, F.Cu at (132.1, 127.5)
- moved C24 172.7 mm to (102.1, 89.4), turned to 180 degrees
- moved R11 121.7 mm to (153.9, 58.2), turned to 270 degrees
- moved C28 109.9 mm to (153.9, 61.7), turned to 270 degrees
- moved R1 108.6 mm to (122.6, 114.6), turned to 90 degrees
- moved R18 107.4 mm to (163.6, 60.5), turned to 270 degrees
- moved R27 102.5 mm to (174.2, 45.0), turned to 90 degrees
- moved R22 99.7 mm to (181.4, 112.3), turned to 90 degrees
- moved R10 97.7 mm to (166.9, 65.0), turned to 180 degrees
- moved R20 97.7 mm to (171.4, 111.0), turned to 270 degrees
- moved R19 97.0 mm to (166.9, 63.0)
- moved R30 93.2 mm to (164.3, 79.5), turned to 270 degrees
- moved R16 92.7 mm to (173.0, 86.1), turned to 180 degrees
- moved R12 91.8 mm to (159.3, 122.7), turned to 90 degrees
- moved C41 91.7 mm to (175.0, 61.0), turned to 270 degrees
- moved R29 89.5 mm to (164.3, 75.9), turned to 270 degrees
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Connections:
- net SHUTDOWN renamed Net-(R3-Pad2)
- J4 pad R: Net-(J4-PadR) -> Net-(C37-Pad2)
- J4 pad T: Net-(J4-PadT) -> Net-(C36-Pad2)
- R27 pad 2: Net-(J4-PadT) -> Net-(C36-Pad2)
- R28 pad 2: Net-(J4-PadR) -> Net-(C37-Pad2)
Routing:
- net +3V3: track 239.8 -> 71.1 mm, vias 6 -> 38
- net RND_BTN: track 0.00 -> 71.1 mm, vias 0 -> 3
- net NEXT_BTN: track 1.38 -> 68.7 mm, vias 1 -> 3
- net PREV_BTN: track 0.00 -> 60.3 mm, vias 0 -> 3
- net SELECT_L: track 0.00 -> 58.0 mm, vias 0 -> 2
- net OPT_BTN: track 1.93 -> 56.5 mm, vias 1 -> 3
- net GND: track 0.00 -> 54.4 mm, vias 5 -> 136
- net SELECT_BTN: track 0.00 -> 54.3 mm, vias 0 -> 3
- net SCK: track 9.37 -> 55.0 mm, vias 2 -> 4
- net MISO: track 15.0 -> 59.0 mm, vias 0 -> 2
- net SS: track 0.00 -> 40.8 mm, vias 0 -> 2
- net +5VA: track 76.5 -> 38.6 mm, vias 2 -> 14
- net MOSI: track 10.3 -> 47.8 mm, vias 2 -> 4
- net SELECT_R: track 0.00 -> 35.5 mm, vias 0 -> 3
- net Net-(C36-Pad2): track 0.00 -> 23.7 mm
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- added copper zone on F.Cu, net +3V3
- added copper zone on In2.Cu, net +3V3
- added copper zone on In2.Cu, net +5VA
- added copper zone on B.Cu, net GND
- added copper zone on In1.Cu, net GND
Other:
- net class Default: clearance 0.2 -> 0.13
- rule trace_clearance: 0.2 -> 0.13
- board text added: "*"
- board text added: "2021"
- board text added: "2021 Aidan Lawrence www.aidanlawrence.com Analog stage schematic courtesy of: KUNOICHI LABS kunoichilabs.dev"
- board text added: "<"
- board text added: ">"
- board text added: "DEBUG"
- board text added: "DIP Switches: YM2612 = ALL LEFT YM3438 = ALL RIGHT"
- board text added: "FLASH"
- board text added: "GND"
- board text added: "JLCJLCJLCJLC"
- board text added: "Kunoichi Analog Stage"
- board text added: "LINE_L"
- board text added: "LINE_R"
- board text added: "M3"
- board text added: "OPA"
- board text added: "OPTION"
- board text added: "PSG MIX"
- board text added: "PWR"
- board text added: "RAM"
- board text added: "RAND"
- board text added: "RESET"
- board text added: "SWD"
- board text added: "Sega Genesis VGM Player"
- board text added: "V1"
- board text added: "VBOOST"
- board text added: "VBUS"
- board text added: "VOLUME"
- board text added: "www.AidanLawrence.com"
