File: MegaBlaster2.sch (KiCad schematic (older format))
At the start: 114 parts, among them J1 USB_B, J2 SWD, J3 Micro_SD_Card, J4 AudioJack3, SW1 SW_SPDT, SW2 SW_Push_Dual, SW3 SW_Push_Dual, SW4 SW_Push_Dual, SW5 SW_Push_Dual, SW6 SW_Push_Dual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

Commit message: Routing
Parts:
- added TP6: TestPoint, TestPoint:TestPoint_Pad_2.0x2.0mm, symbol Connector:TestPoint
Connections:
- net D0: now also U1.44 (PA23); no longer U1.35 (PA16)
- net D1: now also U1.43 (PA22); no longer U1.36 (PA17)
- net D2: now also U1.42 (PA21); no longer U1.37 (PA18)
- net D3: now also U1.41 (PA20); no longer U1.38 (PA19)
- net D4: now also U1.38 (PA19); no longer U1.41 (PA20)
- net D5: now also U1.37 (PA18); no longer U1.42 (PA21)
- net D6: now also U1.36 (PA17); no longer U1.43 (PA22)
- net D7: now also U1.35 (PA16); no longer U1.44 (PA23)
- net GND: now also TP6.1
- net PSG_WE: now also U1.40 (PB17)
- net RAM_CS: now also U1.16 (PA07); no longer U1.60 (PB31)
Changed lines of the file:
@@
 Text GLabel 3450 3850 2    50   Input ~ 0
 SWO
-Text GLabel 2050 3350 0    50   Input ~ 0
+Text GLabel 2050 3450 0    50   Input ~ 0
+D6
+Text GLabel 2050 3550 0    50   Input ~ 0
+D5
+Text GLabel 2050 3650 0    50   Input ~ 0
+D4
+Text GLabel 2050 3750 0    50   Input ~ 0
+D3
+Text GLabel 2050 3850 0    50   Input ~ 0
+D2
+Text GLabel 2050 3950 0    50   Input ~ 0
+D1
+Text GLabel 2050 4050 0    50   Input ~ 0
 D0
-Text GLabel 2050 3450 0    50   Input ~ 0
-D1
-Text GLabel 2050 3550 0    50   Input ~ 0
-D2
-Text GLabel 2050 3650 0    50   Input ~ 0
-D3
-Text GLabel 2050 3750 0    50   Input ~ 0
-D4
-Text GLabel 2050 3850 0    50   Input ~ 0
-D5
-Text GLabel 2050 3950 0    50   Input ~ 0
-D6
-Text GLabel 2050 4050 0    50   Input ~ 0
-D7
 Text GLabel 2050 3250 0    50   Input ~ 0
 SS
@@
 	1    0    0    -1
 $EndComp
-Text GLabel 3450 3950 2    50   Input ~ 0
+Text GLabel 2050 2450 0    50   Input ~ 0
 RAM_CS
 Text GLabel 6950 5800 2    50   Input ~ 0
@@
 	1    0    0    -1
 $EndComp
+$Comp
+L power:GND #PWR088
+U 1 1 5FE2674E
+P 14300 9650
+F 0 "#PWR088" H 14300 9400 50  0001 C CNN
+F 1 "GND" H 14305 9477 50  0000 C CNN
+F 2 "" H 14300 9650 50  0001 C CNN
+F 3 "" H 14300 9650 50  0001 C CNN
+	1    14300 9650
+	1    0    0    -1
+$EndComp
+$Comp
+L Connector:TestPoint TP6
+U 1 1 5FE27B13
+P 14300 9450
+F 0 "TP6" H 14358 9568 50  0000 L CNN
+F 1 "TestPoint" H 14358 9477 50  0000 L CNN
+F 2 "TestPoint:TestPoint_Pad_2.0x2.0mm" H 14500 9450 50  0001 C CNN
+F 3 "~" H 14500 9450 50  0001 C CNN
+	1    14300 9450
+	1    0    0    -1
+$EndComp
+Wire Wire Line
+	14300 9450 14300 9650
+Text GLabel 2050 3350 0    50   Input ~ 0
+D7
+Text GLabel 3450 3550 2    50   Input ~ 0
+PSG_WE
 $EndSCHEMATC

Commit message: Board v1 complete
Parts:
- removed R23, R24: 10R, Resistor_SMD:R_0805_2012Metric, symbol Device:R_Small
- removed SW1: SW_SPDT, Button_Switch_THT:SW_Slide_1P2T_CK_OS102011MS2Q, symbol Switch:SW_SPDT
Connections:
- net at C36.2: now also J4.T, R27.2
- net at C37.2: now also J4.R, R28.2
- net SHUTDOWN: no longer names the net of R3.2, U2.4 (EN)
- no-connect marks 28 -> 27
Changed lines of the file:
@@
 	1    0    0    -1
 $EndComp
-Text GLabel 2900 9650 0    50   Input ~ 0
-SHUTDOWN
-Wire Wire Line
-	2900 9650 3250 9650
-Wire Wire Line
-	3250 9650 3250 9700
-Connection ~ 3450 9700
-$Comp
-L Switch:SW_SPDT SW1
-U 1 1 5FD6F70F
-P 2150 8700
-F 0 "SW1" H 2150 8985 50  0000 C CNN
-F 1 "SW_SPDT" H 2150 8894 50  0000 C CNN
-F 2 "Button_Switch_THT:SW_Slide_1P2T_CK_OS102011MS2Q" H 2150 8700 50  0001 C CNN
-F 3 "~" H 2150 8700 50  0001 C CNN
-	1    2150 8700
-	1    0    0    -1
-$EndComp
-Text GLabel 2350 8600 2    50   Input ~ 0
-SHUTDOWN
-$Comp
-L power:GND #PWR07
-U 1 1 5FD71BF4
-P 1850 8700
-F 0 "#PWR07" H 1850 8450 50  0001 C CNN
-F 1 "GND" H 1855 8527 50  0000 C CNN
-F 2 "" H 1850 8700 50  0001 C CNN
-F 3 "" H 1850 8700 50  0001 C CNN
-	1    1850 8700
-	1    0    0    -1
-$EndComp
-Wire Wire Line
-	1850 8700 1950 8700
-NoConn ~ 2350 8800
 Text GLabel 1150 4750 0    50   Input ~ 0
 RESET
@@
 	0    -1   -1   0
 $EndComp
-Wire Wire Line
-	13500 7450 13650 7450
-$Comp
-L Device:R_Small R23
-U 1 1 601A41B3
-P 13750 7450
-F 0 "R23" V 13554 7450 50  0000 C CNN
-F 1 "10R" V 13645 7450 50  0000 C CNN
-F 2 "Resistor_SMD:R_0805_2012Metric" H 13750 7450 50  0001 C CNN
-F 3 "~" H 13750 7450 50  0001 C CNN
-	1    13750 7450
-	0    1    1    0
-$EndComp
-$Comp
-L Device:R_Small R24
-U 1 1 601A59C3
-P 13750 7750
-F 0 "R24" V 13554 7750 50  0000 C CNN
-F 1 "10R" V 13645 7750 50  0000 C CNN
-F 2 "Resistor_SMD:R_0805_2012Metric" H 13750 7750 50  0001 C CNN
-F 3 "~" H 13750 7750 50  0001 C CNN
-	1    13750 7750
-	0    1    1    0
-$EndComp
-Wire Wire Line
-	13850 7450 14050 7450
-Wire Wire Line
-	13850 7750 14350 7750
 $Comp
 L Device:R_Small R27
@@
 	1    0    0    -1
 $EndComp
-Wire Wire Line
-	3250 9700 3450 9700
 $Comp
 L Connector:USB_B J1
@@
 Text GLabel 3450 3550 2    50   Input ~ 0
 PSG_WE
+Wire Wire Line
+	13500 7450 14050 7450
+Wire Wire Line
+	13650 7750 14350 7750
 $EndSCHEMATC
