File: schematic/MegaBlaster2.kicad_pcb (KiCad board)
At the start: 4 copper layers, 99 x 99 mm, 114 parts, among them J1 USB_B, J2 SWD, J3 Micro_SD_Card, J4 AudioJack3, SW2 SW_Push_Dual, SW3 SW_Push_Dual, SW4 SW_Push_Dual, SW5 SW_Push_Dual, SW6 SW_Push_Dual, SW7 SW_Push_Dual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

Commit message: Menu lib, neopixel removed from pcb, bootloader
Parts:
- removed D2: NeoPixel_THT, LED_SMD:LED_WS2812B_PLCC4_5.0x5.0mm_P3.2mm
Routing:
- net NEOPIX: track 9.41 -> 0.00 mm
- net +3V3: track 71.1 -> 69.9 mm, vias 38 -> 37

Commit message: silkscreen update
Other:
- board text added: "V2"
- board text removed: "V1"

Commit message: PCB Update
Parts:
- added G***: LOGO, Art:FM_2, B.Cu at (133.3, 99.0)
- added G***: LOGO, Art:FM_1, B.Cu at (133.3, 70.4)
- added G***: LOGO, Art:triangle, F.Cu at (86.2, 126.3)
- added G***: LOGO, Art:triangle, F.Cu at (117.2, 126.3)
- added G***: LOGO, Art:triangle, F.Cu at (101.7, 138.8)
- added G***: LOGO, Art:triangle, F.Cu at (101.7, 113.9)
- added R23: 10K, Resistor_SMD:R_0805_2012Metric, F.Cu at (138.2, 99.1)
- moved SW4 2.89 mm to (98.4, 131.1)
- moved SW5 2.89 mm to (107.3, 124.1)
- moved SW6 2.89 mm to (98.4, 117.1)
- moved SW3 2.89 mm to (89.6, 124.1)
- moved SW7 2.89 mm to (98.5, 124.1)
Connections:
- U1 pad 50: Net-(U1-Pad50) -> YM_IRQ
- U8 pad 13: Net-(U8-Pad13) -> YM_IRQ
Routing:
- net YM_IRQ: track 0.00 -> 59.4 mm, vias 0 -> 2
- net PREV_BTN: track 60.3 -> 73.0 mm
- net OPT_BTN: track 56.5 -> 51.6 mm
- net SELECT_BTN: track 54.3 -> 57.8 mm
- net GND: track 54.4 -> 57.6 mm, vias 136 -> 144
- net +3V3: track 69.9 -> 73.1 mm
- net D-: track 55.8 -> 58.2 mm
- net D+: track 56.6 -> 58.9 mm
- net VBOOST: track 79.0 -> 81.0 mm
- net RND_BTN: track 71.1 -> 72.9 mm
- net NEXT_BTN: track 68.7 -> 67.5 mm
- net SCL: track 68.5 -> 69.2 mm
- net SDA: track 69.4 -> 70.1 mm
Other:
- board text added: "...oh and 3 channels of square waves and 1 channel of noise. TY PSG"
- board text removed: "<"
- board text removed: ">"
- board text removed: "OPTION"
- board text removed: "RAND"

Commit message: Schematic cleanup
Routing:
- net D6: track 62.2 -> 56.0 mm
- net GND: vias 144 -> 146
Other:
- board text added: "V2a"
- board text removed: "V2"
