File: schematic/MegaBlaster2.sch (KiCad schematic (older format))
At the start: 112 parts, among them J1 USB_B, J2 SWD, J3 Micro_SD_Card, J4 AudioJack3, SW2 SW_Push_Dual, SW3 SW_Push_Dual, SW4 SW_Push_Dual, SW5 SW_Push_Dual, SW6 SW_Push_Dual, SW7 SW_Push_Dual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

Commit message: Menu lib, neopixel removed from pcb, bootloader
Parts:
- removed D2: NeoPixel_THT, LED_SMD:LED_WS2812B_PLCC4_5.0x5.0mm_P3.2mm, symbol LED:NeoPixel_THT
Connections:
- no-connect marks 27 -> 26
Changed lines of the file:
@@
 Text GLabel 8950 4000 0    50   Input ~ 0
 D7
-$Comp
-L LED:NeoPixel_THT D2
-U 1 1 5FE99965
-P 6500 4650
-F 0 "D2" H 6844 4696 50  0000 L CNN
-F 1 "NeoPixel_THT" H 6844 4605 50  0000 L CNN
-F 2 "LED_SMD:LED_WS2812B_PLCC4_5.0x5.0mm_P3.2mm" H 6550 4350 50  0001 L TNN
-F 3 "https://www.adafruit.com/product/1938" H 6600 4275 50  0001 L TNN
-	1    6500 4650
-	1    0    0    -1
-$EndComp
 Text GLabel 8850 2600 0    50   Input ~ 0
 YM_IC
@@
 Text GLabel 3450 3350 2    50   Input ~ 0
 YM_WR
-Text GLabel 6200 4650 0    50   Input ~ 0
-NEOPIX
-$Comp
-L power:+3V3 #PWR036
-U 1 1 5FECD750
-P 6500 4350
-F 0 "#PWR036" H 6500 4200 50  0001 C CNN
-F 1 "+3V3" H 6515 4523 50  0000 C CNN
-F 2 "" H 6500 4350 50  0001 C CNN
-F 3 "" H 6500 4350 50  0001 C CNN
-	1    6500 4350
-	1    0    0    -1
-$EndComp
-$Comp
-L power:GND #PWR037
-U 1 1 5FECE043
-P 6500 4950
-F 0 "#PWR037" H 6500 4700 50  0001 C CNN
-F 1 "GND" H 6505 4777 50  0000 C CNN
-F 2 "" H 6500 4950 50  0001 C CNN
-F 3 "" H 6500 4950 50  0001 C CNN
-	1    6500 4950
-	1    0    0    -1
-$EndComp
-NoConn ~ 6800 4650
 Text Notes 14300 10250 0    50   ~ 0
 Kunoichi Analog Stage

Commit message: PCB Update
Parts:
- added R23: 10K, Resistor_SMD:R_0805_2012Metric, symbol Device:R_Small
Connections:
- net +3V3: now also R23.1
- net YM_IRQ: now reaches U1.50 (PB23)
- net YM_IRQ: now also U8.13 (IRQ), R23.2
- no-connect marks 26 -> 25
Changed lines of the file:
@@
 YM_IC
 NoConn ~ 8850 2500
-NoConn ~ 9950 2700
 Text GLabel 9950 2600 2    50   Input ~ 0
 YM_CS
@@
 Wire Wire Line
 	13650 7750 14350 7750
+Text GLabel 4250 3750 2    50   Input ~ 0
+YM_IRQ
+Text GLabel 9950 2700 2    50   Input ~ 0
+YM_IRQ
+$Comp
+L Device:R_Small R23
+U 1 1 6006614F
+P 4050 3650
+F 0 "R23" H 4109 3696 50  0000 L CNN
+F 1 "10K" H 4109 3605 50  0000 L CNN
+F 2 "Resistor_SMD:R_0805_2012Metric" H 4050 3650 50  0001 C CNN
+F 3 "~" H 4050 3650 50  0001 C CNN
+	1    4050 3650
+	1    0    0    -1
+$EndComp
+Wire Wire Line
+	3450 3750 4050 3750
+Wire Wire Line
+	4050 3750 4250 3750
+Connection ~ 4050 3750
+$Comp
+L power:+3V3 #PWR07
+U 1 1 6008EE50
+P 4050 3550
+F 0 "#PWR07" H 4050 3400 50  0001 C CNN
+F 1 "+3V3" H 4065 3723 50  0000 C CNN
+F 2 "" H 4050 3550 50  0001 C CNN
+F 3 "" H 4050 3550 50  0001 C CNN
+	1    4050 3550
+	1    0    0    -1
+$EndComp
 $EndSCHEMATC

Commit message: Schematic cleanup
Other:
- note added: "Clock & Sound Chips"
- note added: "I/O"
- note added: "MCU, Flash, RAM"
- note added: "Mixer, Pre-amp, Power Amp"
- note added: "Power"
- note added: "SD"
- moved on the sheet: C1, C10, C11, C12, C13, C14, C15, C16, C17, C18, C19, C2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
